File: rt65b-breakout.kicad_pcb (KiCad board)
At the start: 2 copper layers, 93.2 x 38 mm, 12 parts, among them J1 DIN-7, J3 IEC320-C14

Commit message: added back layer gnd trace
Routing:
- net GND: track 20.4 -> 40.7 mm
Changed lines of the file:
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@@
     (thickness 1.6)
     (drawings 53)
-    (tracks 61)
+    (tracks 63)
     (zones 0)
     (modules 12)
@@
   (layers
     (0 F.Cu signal)
-    (31 B.Cu signal)
+    (31 B.Cu signal hide)
     (32 B.Adhes user)
     (33 F.Adhes user)
@@
     (44 Edge.Cuts user)
     (45 Margin user)
-    (46 B.CrtYd user)
-    (47 F.CrtYd user)
+    (46 B.CrtYd user hide)
+    (47 F.CrtYd user hide)
     (48 B.Fab user)
-    (49 F.Fab user)
+    (49 F.Fab user hide)
   )
   (setup
-    (last_trace_width 2)
+    (last_trace_width 3)
     (user_trace_width 0.5)
     (user_trace_width 1)
@@
   (segment (start 162.75 54) (end 162.75 44.25) (width 3) (layer F.Cu) (net 4))
   (segment (start 170.25 61.5) (end 162.75 54) (width 3) (layer F.Cu) (net 4))
+  (segment (start 162.75 54) (end 162.75 44.25) (width 3) (layer B.Cu) (net 4))
+  (segment (start 170.25 61.5) (end 162.75 54) (width 3) (layer B.Cu) (net 4))
   (segment (start 170.25 66.5) (end 172.75 64) (width 3) (layer F.Cu) (net 5))
   (segment (start 173.75 63) (end 172.75 64) (width 3) (layer F.Cu) (net 5))
